Commit message: add lidar sensor

File: src/first_robot/urdf/gazebo_control.urdf.xacro (robot description, xacro)
@@ -18,4 +18,6 @@
             <publishOdomTF>true</publishOdomTF>
             <publishWheelTF>true</publishWheelTF>
+            <odometryFrame>odom</odometryFrame>
+            <publishTf>true</publishTf>
         </plugin>
     </gazebo>

File: src/first_robot/urdf/lidar.urdf.xacro (robot description, xacro)
@@ -1,4 +1,55 @@
 <?xml version="1.0"?>
-<robot name="my_robot" xmlns:xacro="http://www.ros.org/wiki/xacro">
+<robot xmlns:xacro="http://www.ros.org/wiki/xacro" >
     <joint name="laser_joint" type="fixed">
+        <parent link="chassis"/>
+        <child link="laser_frame"/>
+        <origin xyz="0.1 0 0.175" rpy="0 0 0"/>
+    </joint>
+    <link name="laser_frame">
+        <visual>
+            <geometry>
+                <cylinder radius="0.05" length="0.04"/>
+            </geometry>
+            <material name="red"/>
+        </visual>
+        <collision>
+            <geometry>
+                <cylinder radius="0.05" length="0.04"/>
+            </geometry>
+        </collision>
+        <xacro:inertial_cylinder mass="0.1" length="0.04" radius="0.05">
+            <origin xyz="0 0 0" rpy="0 0 0"/>
+        </xacro:inertial_cylinder>
+    </link>
+    <gazebo reference="laser_frame">
+        <material>Gazebo/Red</material>
+        <sensor name="laser" type="ray">
+            <pose> 0 0 0 0 0 0 </pose>
+            <always_on>true</always_on>
+            <visualize>true</visualize>
+            <update_rate>10</update_rate>
+            <ray>
+                <scan>
+                    <horizontal>
+                        <samples>360</samples>
+                        <resolution>1</resolution>
+                        <min_angle>-3.14</min_angle>
+                        <max_angle>3.14</max_angle>
+                    </horizontal>
+                </scan>
+                <range>
+                    <min>0.3</min>
+                    <max>12</max>
+                    <resolution>0.01</resolution>
+                </range>
+            </ray>
+            <plugin name="laser_controller" filename="libgazebo_ros_laser.so">
+                <topicName>scan</topicName>
+                <frameName>laser_frame</frameName>
+            </plugin>
+        </sensor>
+    </gazebo>
+    <material name="red">
+        <color rgba="1 0 0 1"/>
+    </material>
 </robot>

File: src/first_robot/urdf/v2_robot.urdf.xacro (robot description, xacro)
@@ -3,3 +3,4 @@
       <xacro:include filename="robot_core.urdf.xacro" />
       <xacro:include filename="gazebo_control.urdf.xacro" />
+      <xacro:include filename="lidar.urdf.xacro" />
 </robot>

Commit message: added imu sensor and adde base_footprint link

File: src/first_robot/urdf/gazebo_control.urdf.xacro (robot description, xacro)
@@ -13,9 +13,9 @@
             <commandTopic>cmd_vel</commandTopic>
             <odometryTopic>odom</odometryTopic>
-            <robotBaseFrame>base_link</robotBaseFrame>
+            <robotBaseFrame>base_footprint</robotBaseFrame>
             <!-- TF / Odom -->
             <publishOdom>true</publishOdom>
             <publishOdomTF>true</publishOdomTF>
-            <publishWheelTF>true</publishWheelTF>
+            <publishWheelTF>false</publishWheelTF>
             <odometryFrame>odom</odometryFrame>
             <publishTf>true</publishTf>

File: src/first_robot/urdf/imu.urdf.xacro (robot description, xacro)
@@ -4,21 +4,31 @@
         <parent link="chassis"/>
         <child link="imu_frame"/>
-        <origin xyz="0.4 0 0.175" rpy="0 0 0"/>
+        <origin xyz="0.15 0 0.175" rpy="0 0 0"/>
     </joint>
-    <link name="imu_frame_frame">
+    <link name="imu_frame">
             <visual>
                 <geometry>
-                    <cylinder radius="0.05" length="0.04"/>
+                    <cylinder radius="0.02" length="0.03"/>
                 </geometry>
-                <material name="red"/>
+                <material name="blue"/>
             </visual>
             <collision>
                 <geometry>
-                    <cylinder radius="0.05" length="0.04"/>
+                    <cylinder radius="0.02" length="0.03"/>
                 </geometry>
             </collision>
-            <xacro:inertial_cylinder mass="0.1" length="0.04" radius="0.05">
+            <xacro:inertial_cylinder mass="0.1" length="0.03" radius="0.02">
                 <origin xyz="0 0 0" rpy="0 0 0"/>
             </xacro:inertial_cylinder>
     </link>
-<robot>
+  <gazebo>
+    <plugin name="imu_plugin" filename="libgazebo_ros_imu.so">
+      <alwaysOn>true</alwaysOn>
+      <bodyName>base_link</bodyName>
+      <topicName>imu</topicName>
+      <serviceName>imu_service</serviceName>
+      <gaussianNoise>0.0</gaussianNoise>
+      <updateRate>10.0</updateRate>
+    </plugin>
+  </gazebo>
+</robot>

File: src/first_robot/urdf/lidar.urdf.xacro (robot description, xacro)
@@ -4,5 +4,5 @@
         <parent link="chassis"/>
         <child link="laser_frame"/>
-        <origin xyz="0.1 0 0.175" rpy="0 0 0"/>
+        <origin xyz="0.25 0 0.175" rpy="0 0 0"/>
     </joint>
     <link name="laser_frame">

File: src/first_robot/urdf/robot_core.urdf.xacro (robot description, xacro)
@@ -14,4 +14,12 @@
         <color rgba="0 0 0 1"/>
     </material>
+<!-- BASE FOOTPRINT -->
+    <link name="base_footprint"/>
+    <joint name="base_footprint_joint" type="fixed">
+        <parent link="base_footprint"/>
+        <child link="base_link"/>
+        <origin xyz="0 0 0.05" rpy="0 0 0"/> <!-- 0.05 επειδή η ακτίνα των τροχών είναι 0.05 -->
+    </joint>
+    <!-- BASE LINK -->
     <link name="base_link">
     </link>

File: src/first_robot/urdf/v2_robot.urdf.xacro (robot description, xacro)
@@ -5,3 +5,4 @@
       <xacro:include filename="lidar.urdf.xacro" />
       <xacro:include filename="camera.urdf.xacro" />
+      <xacro:include filename="imu.urdf.xacro" />
 </robot>

Commit message: added gps module, changed diff_controller to read parameters from yaml file and implemented local EKF

File: src/first_robot/urdf/gazebo_control.urdf.xacro (robot description, xacro)
@@ -2,23 +2,57 @@
 <robot name="my_robot" xmlns:xacro="http://www.ros.org/wiki/xacro">
     <gazebo>
-        <plugin name="diff_drive" filename="libgazebo_ros_diff_drive.so">
-            <!-- Required -->
-            <leftJoint>left_wheel_joint</leftJoint>
-            <rightJoint>right_wheel_joint</rightJoint>
-            <wheelSeparation>0.35</wheelSeparation>
-            <wheelDiameter>0.1</wheelDiameter>
-            <wheelTorque>200</wheelTorque>
-            <wheelAcceleration>10.0</wheelAcceleration>
-            <!-- Topics -->
-            <commandTopic>cmd_vel</commandTopic>
-            <odometryTopic>odom</odometryTopic>
-            <robotBaseFrame>base_footprint</robotBaseFrame>
-            <!-- TF / Odom -->
-            <publishOdom>true</publishOdom>
-            <publishOdomTF>true</publishOdomTF>
-            <publishWheelTF>false</publishWheelTF>
-            <odometryFrame>odom</odometryFrame>
-            <publishTf>true</publishTf>
+        <plugin name="gazebo_ros_control" filename="libgazebo_ros_control.so">
+            <robotNamespace></robotNamespace>
+            <robotSimType>gazebo_ros_control/DefaultRobotHWSim</robotSimType>
+            <legacyModeNS>false</legacyModeNS>
         </plugin>
     </gazebo>
+    <gazebo>
+        <plugin name="p3d_base_controller" filename="libgazebo_ros_p3d.so">
+            <alwaysOn>true</alwaysOn>
+            <updateRate>100.0</updateRate>
+            <bodyName>base_footprint</bodyName>
+            <topicName>ground_truth</topicName>
+            <gaussianNoise>0.0</gaussianNoise>
+            <frameName>world</frameName>
+            <xyzOffsets>0 0 0</xyzOffsets>
+            <rpyOffsets>0 0 0</rpyOffsets>
+        </plugin>
+    </gazebo>
+    <transmission name="left_wheel_trans">
+        <type>transmission_interface/SimpleTransmission</type>
+        <joint name="left_wheel_joint">
+            <hardwareInterface>hardware_interface/VelocityJointInterface</hardwareInterface>
+        </joint>
+        <actuator name="left_wheel_motor">
+            <mechanicalReduction>1</mechanicalReduction>
+            <hardwareInterface>hardware_interface/VelocityJointInterface</hardwareInterface>
+        </actuator>
+    </transmission>
+    <transmission name="right_wheel_trans">
+        <type>transmission_interface/SimpleTransmission</type>
+        <joint name="right_wheel_joint">
+            <hardwareInterface>hardware_interface/VelocityJointInterface</hardwareInterface>
+        </joint>
+        <actuator name="right_wheel_motor">
+            <mechanicalReduction>1</mechanicalReduction>
+            <hardwareInterface>hardware_interface/VelocityJointInterface</hardwareInterface>
+        </actuator>
+    </transmission>
+    <gazebo reference="$right_wheel_link">
+        <kp>100000000</kp>
+        <kd>1</kd>
+        <mu1>200</mu1>
+        <mu2>10</mu2>
+        <maxVel>4.0</maxVel>
+        <minDepth>0.01</minDepth>
+    </gazebo>
+    <gazebo reference="left_wheel_link">
+        <kp>100000000</kp>
+        <kd>1</kd>
+        <mu1>200</mu1>
+        <mu2>10</mu2>
+        <maxVel>4.0</maxVel>
+        <minDepth>0.01</minDepth>
+    </gazebo>
 </robot>

File: src/first_robot/urdf/imu.urdf.xacro (robot description, xacro)
@@ -4,30 +4,29 @@
         <parent link="chassis"/>
         <child link="imu_frame"/>
-        <origin xyz="0.15 0 0.175" rpy="0 0 0"/>
     </joint>
-    <link name="imu_frame">
+            <link name="imu_frame">
+            <inertial>
+                <origin xyz="0.0 0 0.01" rpy="0 0 0" />
+                <mass value="0.005" />
+                <inertia  ixx="8.333333333333334e-10" ixy = "0" ixz = "0"
+                    iyy="8.333333333333334e-10" iyz = "0"
+                    izz="8.333333333333334e-10"
+                    />
+            </inertial>
             <visual>
+                <origin rpy="0 0 0" xyz="0 0 0"/>
                 <geometry>
-                    <cylinder radius="0.02" length="0.03"/>
+                    <box size="0.001 0.001 0.001"/>
                 </geometry>
-                <material name="blue"/>
             </visual>
-            <collision>
-                <geometry>
-                    <cylinder radius="0.02" length="0.03"/>
-                </geometry>
-            </collision>
-            <xacro:inertial_cylinder mass="0.1" length="0.03" radius="0.02">
-                <origin xyz="0 0 0" rpy="0 0 0"/>
-            </xacro:inertial_cylinder>
-    </link>
+        </link>
   <gazebo>
     <plugin name="imu_plugin" filename="libgazebo_ros_imu.so">
       <alwaysOn>true</alwaysOn>
-      <bodyName>base_link</bodyName>
+      <bodyName>base_footprint</bodyName>
       <topicName>imu</topicName>
       <serviceName>imu_service</serviceName>
       <gaussianNoise>0.0</gaussianNoise>
-      <updateRate>10.0</updateRate>
+      <updateRate>100.0</updateRate>
     </plugin>
   </gazebo>

File: src/first_robot/urdf/robot_core.urdf.xacro (robot description, xacro)
@@ -22,6 +22,5 @@
     </joint>
     <!-- BASE LINK -->
-    <link name="base_link">
-    </link>
+    <link name="base_link"/>
     <joint name="chassis_joint" type="fixed">
         <parent link="base_link"/>

File: src/first_robot/urdf/v2_robot.urdf.xacro (robot description, xacro)
@@ -3,6 +3,7 @@
       <xacro:include filename="robot_core.urdf.xacro" />
       <xacro:include filename="gazebo_control.urdf.xacro" />
-      <xacro:include filename="lidar.urdf.xacro" />
+      <!-- <xacro:include filename="lidar.urdf.xacro" /> -->
       <xacro:include filename="camera.urdf.xacro" />
       <xacro:include filename="imu.urdf.xacro" />
+      <xacro:include filename="gps.urdf.xacro" />
 </robot>
